Commit message: Config simulation part

File: rm_simulation/ma_sentry_urdf/urdf/ma_sentry_urdf.urdf (robot description, URDF)
Before this commit: robot 车架总成, 6 links, 5 joints
Links:
- link 1_Link: geometry collision mesh filename=package://ma_sentry_urdf/meshes/1_Link.STL; visual mesh filename=package://ma_sentry_urdf/meshes/1_Link.STL
- link 2_Link: geometry collision mesh filename=package://ma_sentry_urdf/meshes/2_Link.STL; visual mesh filename=package://ma_sentry_urdf/meshes/2_Link.STL
- link 3_Link: geometry collision mesh filename=package://ma_sentry_urdf/meshes/3_Link.STL; visual mesh filename=package://ma_sentry_urdf/meshes/3_Link.STL
- link 4_Link: geometry collision mesh filename=package://ma_sentry_urdf/meshes/4_Link.STL; visual mesh filename=package://ma_sentry_urdf/meshes/4_Link.STL
- link 5_Link: geometry collision mesh filename=package://ma_sentry_urdf/meshes/5_Link.STL; visual mesh filename=package://ma_sentry_urdf/meshes/5_Link.STL
- link base_link: geometry collision mesh filename=package://ma_sentry_urdf/meshes/base_link.STL; visual mesh filename=package://ma_sentry_urdf/meshes/base_link.STL

Commit message: Add MA sentry urdf

File: rm_simulation/ma_sentry_urdf/urdf/ma_sentry_urdf.urdf (robot description, URDF)
Before this commit: robot ma_sentry_urdf, 7 links, 6 joints
Links:
- removed link 1_Link
- removed link 2_Link
- removed link 3_Link
- removed link 4_Link
- removed link 5_Link
- added link gimbal_Link, mass 2.73797674659914; collision mesh filename=package://ma_sentry_urdf/meshes/5_Link.STL; visual mesh filename=package://ma_sentry_urdf/meshes/5_Link.STL
- added link left_back_wheel_Link, mass 0.436812880165245; collision mesh filename=package://ma_sentry_urdf/meshes/1_Link.STL; visual mesh filename=package://ma_sentry_urdf/meshes/1_Link.STL
- added link left_front_wheel_Link, mass 0.332440985195605; collision mesh filename=package://ma_sentry_urdf/meshes/1_Link.STL; visual mesh filename=package://ma_sentry_urdf/meshes/1_Link.STL
- added link right_back_wheel_Link, mass 0.405088777295711; collision mesh filename=package://ma_sentry_urdf/meshes/1_Link.STL; visual mesh filename=package://ma_sentry_urdf/meshes/1_Link.STL
- added link right_front_wheel_Link, mass 0.272373357196352; collision mesh filename=package://ma_sentry_urdf/meshes/1_Link.STL; visual mesh filename=package://ma_sentry_urdf/meshes/1_Link.STL
Joints:
- joint 1: child 1_Link -> left_front_wheel_Link
- joint 2: child 2_Link -> right_front_wheel_Link
- joint 3: child 3_Link -> right_back_wheel_Link
- joint 4: child 4_Link -> left_back_wheel_Link
- joint 5: child 5_Link -> gimbal_Link
