Commit message: Add MA sentry urdf

File: ma_sentry_bringup/urdf/chassis.urdf.xacro (robot description, xacro)
@@ -1,4 +1,4 @@
 <robot xmlns:xacro="http://www.ros.org/wiki/xacro">
-    <xacro:include filename="$(find rm_description)/urdf/common/omni_wheel.urdf.xacro"/>
+    <xacro:include filename="$(find ma_sentry_bringup)/urdf/common/omni_wheel.urdf.xacro"/>
     <!-- https://upload.wikimedia.org/wikipedia/commons/5/52/Wheelbase_and_Track.png -->
     <xacro:property name="chassis_radius" value="0.196"/>
@@ -9,11 +9,12 @@
                 <mass value="12.326"/>
                 <origin xyz="-0.000932  -0.000668  -0.01"/>
-                <inertia ixx="1.924e-1" ixy="-6.458e-4" ixz="5.951352e-3" iyy="2.473e-1"
-                         iyz="-7.22e-4" izz="3.187e-1"/>
+                <inertia ixx="1.924e-1" ixy="-6.458e-4" ixz="5.951352e-3"
+                         iyy="2.473e-1" iyz="-7.22e-4"
+                         izz="3.187e-1"/>
             </inertial>
             <visual>
                 <origin xyz="0 0 0" rpy="0 0 0"/>
                 <geometry>
-                    <mesh filename="package://rm_description/meshes/standard/base.stl" scale="0.001 0.001 0.001"/>
+                    <mesh filename="package://ma_sentry_bringup/meshes/base.stl" scale="0.001 0.001 0.001"/>
                 </geometry>
             </visual>

File: ma_sentry_bringup/urdf/ma_sentry.urdf.xacro (robot description, xacro)
@@ -2,7 +2,7 @@
 <robot xmlns:xacro="http://www.ros.org/wiki/xacro" name="sentry">
     <xacro:arg name="load_chassis" default="true"/>
-    <xacro:arg name="load_gimbal" default="true"/>
-    <xacro:arg name="load_shooter" default="true"/>
-    <xacro:arg name="use_simulation" default="true"/>
+    <xacro:arg name="load_gimbal" default="false"/>
+    <xacro:arg name="load_shooter" default="false"/>
+    <xacro:arg name="use_simulation" default="false"/>
     <xacro:arg name="roller_type" default="realistic"/>
     <xacro:if value="$(arg load_chassis)">
@@ -18,5 +18,5 @@
     </xacro:if>
     <xacro:if value="$(arg load_gimbal)">
-        <xacro:include filename="$(find ma_sentry_bringup)/urdf/standard/gimbal.urdf.xacro"/>
+        <xacro:include filename="$(find ma_sentry_bringup)/urdf/gimbal.urdf.xacro"/>
         <xacro:include filename="$(find ma_sentry_bringup)/urdf/sentry/gimbal.transmission.urdf.xacro"/>
         <xacro:gimbal simulation="$(arg use_simulation)"/>

Commit message: Add rmuc playground simulation

File: ma_sentry_bringup/urdf/chassis.urdf.xacro (robot description, xacro)
@@ -16,5 +16,5 @@
                 <origin xyz="0 0 0" rpy="0 0 0"/>
                 <geometry>
-                    <mesh filename="package://ma_sentry_bringup/meshes/base.stl" scale="0.001 0.001 0.001"/>
+                    <mesh filename="package://ma_sentry_bringup/meshes/base.stl" scale="0.1 0.1 0.1"/>
                 </geometry>
             </visual>

File: ma_sentry_bringup/urdf/common/omni_wheel.urdf.xacro (robot description, xacro)
@@ -59,5 +59,5 @@
             <visual>
                 <geometry>
-                    <mesh filename="package://ma_sentry_bringup/meshes/common/omni_wheel.stl"
+                    <mesh filename="package://ma_sentry_bringup/meshes/omni_wheel.stl"
                           scale="0.001 0.001 0.001"/>
                 </geometry>

File: ma_sentry_bringup/urdf/ma_sentry.urdf.xacro (robot description, xacro)
@@ -4,5 +4,5 @@
     <xacro:arg name="load_gimbal" default="false"/>
     <xacro:arg name="load_shooter" default="false"/>
-    <xacro:arg name="use_simulation" default="false"/>
+    <xacro:arg name="use_simulation" default="true" />
     <xacro:arg name="roller_type" default="realistic"/>
     <xacro:if value="$(arg load_chassis)">
@@ -10,10 +10,6 @@
         <xacro:chassis roller_type="$(arg roller_type)"/>
         <xacro:include filename="$(find ma_sentry_bringup)/urdf/imu.urdf.xacro"/>
-        <xacro:IMU connected_to="base_link" imu_name="base_imu" simulation="true"
+        <xacro:IMU connected_to="base_link" imu_name="base_imu"
                    xyz="0.065 0.12 0.07"/>
-        <xacro:include filename="$(find ma_sentry_bringup)/urdf/realsense_l515.urdf.xacro"/>
-        <xacro:realsense_l515 connected_to="base_link" realsense_name="base_realsense"
-                              simulation="$(arg use_simulation)"
-                              xyz="0.228618 0 0.10845" rpy="0 0 0"/>
     </xacro:if>
     <xacro:if value="$(arg load_gimbal)">
