Commit message: Change octomap_server launch file

File: rm_simulation/ma_simulation/urdf/mecanum_base.xacro (robot description, xacro)
@@ -1,5 +1,5 @@
 <?xml version="1.0" ?>
 <robot name="mecanum_base" xmlns:xacro="http://www.ros.org/wiki/xacro">
-    <!--<xacro:include filename="$(find sentry_gazebo)/urdf/sc.plugins.xacro" />-->
+    <!--<xacro:include filename="$(find ma_simulation)/urdf/sc.plugins.xacro" />-->
     <material name="blue">
         <color rgba="0 0 0.8 1"/>
@@ -32,5 +32,5 @@
                 <origin rpy="0 0 0" xyz="0 0 0"/>
                 <geometry>
-                    <mesh filename="package://sentry_gazebo/meshes/base_link.stl" scale="0.001 0.001 0.001"/>
+                    <mesh filename="package://ma_simulation/meshes/base_link.stl" scale="0.001 0.001 0.001"/>
                 </geometry>
             </collision>
@@ -39,5 +39,5 @@
                 <origin rpy="0 0 0" xyz="0 0 0"/>
                 <geometry>
-                    <mesh filename="package://sentry_gazebo/meshes/base_link.stl" scale="0.001 0.001 0.001"/>
+                    <mesh filename="package://ma_simulation/meshes/base_link.stl" scale="0.001 0.001 0.001"/>
                 </geometry>
                 <material name="base_link">
@@ -70,11 +70,11 @@
                 <origin xyz="0 0 -0.07625" rpy="0 0 -1.57"/>
                 <geometry>
-                    <mesh filename="package://sentry_gazebo/meshes/mecanum_right_hands.stl" scale="0.001 0.001 0.001"/>
-                </geometry>
-            </collision>
-            <visual>
-                <origin xyz="0 0 -0.07625" rpy="0 0 -1.57"/>
-                <geometry>
-                    <mesh filename="package://sentry_gazebo/meshes/mecanum_right_hands.stl" scale="0.001 0.001 0.001"/>
+                    <mesh filename="package://ma_simulation/meshes/mecanum_right_hands.stl" scale="0.001 0.001 0.001"/>
+                </geometry>
+            </collision>
+            <visual>
+                <origin xyz="0 0 -0.07625" rpy="0 0 -1.57"/>
+                <geometry>
+                    <mesh filename="package://ma_simulation/meshes/mecanum_right_hands.stl" scale="0.001 0.001 0.001"/>
                 </geometry>
                 <material name="wheels">
@@ -102,11 +102,11 @@
                 <origin xyz="0 0 -0.07625" rpy="0 0 -1.57"/>
                 <geometry>
-                    <mesh filename="package://sentry_gazebo/meshes/mecanum_left_hands.stl" scale="0.001 0.001 0.001"/>
-                </geometry>
-            </collision>
-            <visual>
-                <origin xyz="0 0 -0.07625" rpy="0 0 -1.57"/>
-                <geometry>
-                    <mesh filename="package://sentry_gazebo/meshes/mecanum_left_hands.stl" scale="0.001 0.001 0.001"/>
+                    <mesh filename="package://ma_simulation/meshes/mecanum_left_hands.stl" scale="0.001 0.001 0.001"/>
+                </geometry>
+            </collision>
+            <visual>
+                <origin xyz="0 0 -0.07625" rpy="0 0 -1.57"/>
+                <geometry>
+                    <mesh filename="package://ma_simulation/meshes/mecanum_left_hands.stl" scale="0.001 0.001 0.001"/>
                 </geometry>
                 <material name="wheels">
@@ -134,11 +134,11 @@
                 <origin xyz="0 0 -0.07625" rpy="0 0 -1.57"/>
                 <geometry>
-                    <mesh filename="package://sentry_gazebo/meshes/mecanum_left_hands.stl" scale="0.001 0.001 0.001"/>
-                </geometry>
-            </collision>
-            <visual>
-                <origin xyz="0 0 -0.07625" rpy="0 0 -1.57"/>
-                <geometry>
-                    <mesh filename="package://sentry_gazebo/meshes/mecanum_left_hands.stl" scale="0.001 0.001 0.001"/>
+                    <mesh filename="package://ma_simulation/meshes/mecanum_left_hands.stl" scale="0.001 0.001 0.001"/>
+                </geometry>
+            </collision>
+            <visual>
+                <origin xyz="0 0 -0.07625" rpy="0 0 -1.57"/>
+                <geometry>
+                    <mesh filename="package://ma_simulation/meshes/mecanum_left_hands.stl" scale="0.001 0.001 0.001"/>
                 </geometry>
                 <material name="wheels">
@@ -166,11 +166,11 @@
                 <origin xyz="0 0 -0.07625" rpy="0 0 -1.57"/>
                 <geometry>
-                    <mesh filename="package://sentry_gazebo/meshes/mecanum_right_hands.stl" scale="0.001 0.001 0.001"/>
-                </geometry>
-            </collision>
-            <visual>
-                <origin xyz="0 0 -0.07625" rpy="0 0 -1.57"/>
-                <geometry>
-                    <mesh filename="package://sentry_gazebo/meshes/mecanum_right_hands.stl" scale="0.001 0.001 0.001"/>
+                    <mesh filename="package://ma_simulation/meshes/mecanum_right_hands.stl" scale="0.001 0.001 0.001"/>
+                </geometry>
+            </collision>
+            <visual>
+                <origin xyz="0 0 -0.07625" rpy="0 0 -1.57"/>
+                <geometry>
+                    <mesh filename="package://ma_simulation/meshes/mecanum_right_hands.stl" scale="0.001 0.001 0.001"/>
                 </geometry>
                 <material name="wheels">
@@ -213,5 +213,5 @@
       <origin xyz="0 0 0.1" rpy="0 0 0" />
   </xacro:VLP-16>
-  <xacro:include filename="$(find sentry_gazebo)/urdf/camera.urdf.xacro"/>
+  <xacro:include filename="$(find ma_simulation)/urdf/camera.urdf.xacro"/>
   <!-- <xacro:camera parent="base_link">
       <origin xyz="0.1 0 0" rpy="0 0 0" />
