Commit message: Add 2d simulation

File: rm_simulation/ma_simulation/urdf/rmus_map_2.urdf (robot description, URDF)
Before this commit: robot simple_meca_car, 1 links, 0 joints
Links:
- link base_link: geometry collision mesh filename=package://ma_simulation/meshes/base_link.stl; visual mesh filename=package://ma_simulation/meshes/base_link.stl

File: rm_simulation/ma_simulation/urdf/waking_robot.xacro (robot description, xacro)
@@ -244,5 +244,5 @@
       <origin xyz="0 0 0" rpy="0 0 0"/>
       <geometry>
-        <mesh filename="package://simple_meca_car/meshes/hokuyo.dae"/>
+        <mesh filename="package://ma_simulation/meshes/hokuyo.dae"/>
       </geometry>
     </visual>
