Commit message: Add 2d simulation localization

File: rm_simulation/ma_simulation/urdf/waking_robot.xacro (robot description, xacro)
@@ -14,6 +14,4 @@
                </inertial>
 	</xacro:macro>
-    <link name="dummy">
-    </link>
 	<link name="base_footprint">
    		<visual>
@@ -25,8 +23,4 @@
 		<xacro:default_inertial mass="0.0001"/>
  	</link>
-   <joint name="dummy_joint" type="fixed">
-     <parent link="dummy"/>
-     <child link="base_footprint"/>
-   </joint>
 <!--  	<xacro:include filename="$(find nav_sim)/urdf/robot.gazebo" />  -->
 	<gazebo reference="base_footprint">
