Commit message: Add files via upload

File: rm_simulation/ma_simulation/urdf/ma_2d_robot.xacro (robot description, xacro)
@@ -225,8 +225,8 @@
     <parent link="base_link"/>
     <axis xyz="0 1 0" />
-    <child link="laser_frame"/>
+    <child link="laser"/>
   </joint>
   <!-- Hokuyo Laser -->
-  <link name="laser_frame">
+  <link name="laser">
     <collision>
       <origin xyz="0 0 0" rpy="0 0 0"/>
